File: Hardware/Soft_Power_Switch.kicad_pcb (KiCad board)
At the start: 2 copper layers, 25.4 x 25.4 mm, 63 parts, among them J1 JST_2mm_LiPo, J2 JST_2mm_LiPo, J3 Conn_01x06, Q1 BSS138, Q2 BSS138, Q3 SIL2308, SW1 SMD_5.2x5.2mm_h2.5mm, U2 SN74LVC1G14DCK, U3 SN74LVC1G17DCK, U4 SN74LVC1G175DCK

Commit message: Add panel. Single PCB gerbers moved into Production_Single_PCB
Other:
- board text added: "Solder Mask: Red"
- board text removed: "Solder Mask: Black"
Changed lines of the file:
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@@
 		(title "SparkX Soft Power Switch Mk2")
 		(date "2024-03-13")
-		(rev "v01")
+		(rev "v10")
 		(comment 1 "Designed by: Paul Clark")
 	)
@@
 		(fp_arc
 			(start 0.762 -1.016)
-			(mid 1.08529 -0.88209)
+			(mid 1.085289 -0.882089)
 			(end 1.2192 -0.5588)
 			(stroke
@@
 		(fp_arc
 			(start 0.762 -1.016)
-			(mid 1.08529 -0.88209)
+			(mid 1.085289 -0.882089)
 			(end 1.2192 -0.5588)
 			(stroke
@@
 		)
 	)
-	(gr_text "Solder Mask: Black"
+	(gr_text "Solder Mask: Red"
 		(at 196.264108 179.705 0)
 		(layer "F.Fab")
@@
 		)
 		(height -6.401727)
-		(gr_text "1000 mils"
+		(gr_text "25.4 mm"
 			(at 128.27 91.56 0)
 			(layer "Dwgs.User")
@@
 		)
 		(height 2.54)
-		(gr_text "50 mils"
+		(gr_text "1.3 mm"
 			(at 142.36 123.825 90)
 			(layer "Dwgs.User")
@@
 		)
 		(height 2.54)
-		(gr_text "250 mils"
+		(gr_text "6.3 mm"
 			(at 118.745 125.85 0)
 			(layer "Dwgs.User")
@@
 		)
 		(height -6.35)
-		(gr_text "1000 mils"
+		(gr_text "25.4 mm"
 			(at 108.07 111.76 90)
 			(layer "Dwgs.User")
